File: BantamOnOffSwitchGroup.kicad_sch (KiCad schematic)
At the start: 4 parts, among them J1 Conn_01x02_Male, J2 Conn_01x04_Male, SW1 SW_Push_DPDT

Commit message: gbr and drill files created
Other:
- company: (none) -> RoboWidgets
- title: (none) -> Bantamp Power Switch Group
Changed lines of the file:
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@@
 	(generator "eeschema")
 	(generator_version "8.0")
-	(paper "A4")
+	(paper "A")
+	(title_block
+		(title "Bantamp Power Switch Group")
+		(date "2024-03-06")
+		(rev "1")
+		(company "RoboWidgets")
+	)
 	(junction
 		(at 148.336 79.502)
